Commit message: ros2 control done (error fixed)

File: description/robot_core.xacro (robot description, xacro)
@@ -55,11 +55,10 @@
        <!-- All Wheel links and joints -->
     <xacro:macro name="wheel" params="name x y z">
-        <joint name="${name}_wheel_joint" type="continuous">
-            <origin xyz="${x} ${y} ${z}" rpy="-${pi/2} 0.0 0.0"/>
-            <parent link="chassis"/>
-            <child link="${name}_wheel"/>
-            <limit effort="1000.0" velocity="5.0"/>
-            <axis xyz="0.0 0.0 1"/>
-        </joint>
+    <joint name="${name}_wheel_joint" type="continuous">
+        <origin xyz="${x} ${y} ${z}" rpy="-${pi/2} 0.0 0.0"/>
+        <parent link="chassis"/>
+        <child link="${name}_wheel"/>
+        <axis xyz="0.0 0.0 1"/>
+    </joint>
         <link name="${name}_wheel">
             <visual name="">
@@ -82,4 +81,14 @@
             </xacro:inertial_cylinder>
         </link>
+            <transmission name="${name}_trans">
+        <type>transmission_interface/SimpleTransmission</type>
+        <joint name="${name}_wheel_joint">
+            <hardwareInterface>VelocityJointInterface</hardwareInterface>
+        </joint>
+        <actuator name="${name}_motor">
+            <hardwareInterface>VelocityJointInterface</hardwareInterface>
+            <mechanicalReduction>1</mechanicalReduction>
+        </actuator>
+    </transmission>
     </xacro:macro>
     <!-- Wheel Creating using macros -->

File: description/ros2_control.xacro (robot description, xacro)
@@ -1,52 +1,46 @@
 <?xml version="1.0"?>
 <robot xmlns:xacro="http://www.ros.org/wiki/xacro">
-  <!-- MACRO DEFINITION -->
-  <xacro:macro name="wheel_transmission" params="name">
-    <transmission name="${name}_trans">
-      <type>transmission_interface/SimpleTransmission</type>
-      <joint name="${name}_wheel_joint">
-        <hardwareInterface>hardware_interface/VelocityJointInterface</hardwareInterface>
-      </joint>
-      <actuator name="${name}_motor">
-        <hardwareInterface>hardware_interface/VelocityJointInterface</hardwareInterface>
-        <mechanicalReduction>1</mechanicalReduction>
-      </actuator>
-    </transmission>
-  </xacro:macro>
-  <!-- USE MACRO FOR ALL WHEELS -->
-  <xacro:wheel_transmission name="front_left"/>
-  <xacro:wheel_transmission name="front_right"/>
-  <xacro:wheel_transmission name="rear_left"/>
-  <xacro:wheel_transmission name="rear_right"/>
-  <!-- ROS2 CONTROL -->
-  <ros2_control name="GazeboSystem" type="system">
-    <hardware>
-      <plugin>gazebo_ros2_control/GazeboSystem</plugin>
-    </hardware>
-    <joint name="front_left_wheel_joint">
-      <command_interface name="velocity"/>
-      <state_interface name="position"/>
-      <state_interface name="velocity"/>
-    </joint>
-    <joint name="front_right_wheel_joint">
-      <command_interface name="velocity"/>
-      <state_interface name="position"/>
-      <state_interface name="velocity"/>
-    </joint>
-    <joint name="rear_left_wheel_joint">
-      <command_interface name="velocity"/>
-      <state_interface name="position"/>
-      <state_interface name="velocity"/>
-    </joint>
-    <joint name="rear_right_wheel_joint">
-      <command_interface name="velocity"/>
-      <state_interface name="position"/>
-      <state_interface name="velocity"/>
-    </joint>
-  </ros2_control>
-  <gazebo>
-    <plugin name="gazebo_ros2_control" filename="libgazebo_ros2_control.so">
-      <parameters>$(find synhive_robot)/config/my_controllers.yaml</parameters>
-    </plugin>
-  </gazebo>
+    <ros2_control name="GazeboSystem" type="system">
+        <hardware>
+            <plugin>gazebo_ros2_control/GazeboSystem</plugin>
+        </hardware>
+        <!-- Add all 4 wheel joints -->
+        <joint name="front_left_wheel_joint">
+            <command_interface name="velocity">
+                <param name="min">-10</param>
+                <param name="max">10</param>
+            </command_interface>
+            <state_interface name="position"/>
+            <state_interface name="velocity"/>
+        </joint>
+        <joint name="rear_left_wheel_joint">
+            <command_interface name="velocity">
+                <param name="min">-10</param>
+                <param name="max">10</param>
+            </command_interface>
+            <state_interface name="position"/>
+            <state_interface name="velocity"/>
+        </joint>
+        <joint name="front_right_wheel_joint">
+            <command_interface name="velocity">
+                <param name="min">-10</param>
+                <param name="max">10</param>
+            </command_interface>
+            <state_interface name="position"/>
+            <state_interface name="velocity"/>
+        </joint>
+        <joint name="rear_right_wheel_joint">
+            <command_interface name="velocity">
+                <param name="min">-10</param>
+                <param name="max">10</param>
+            </command_interface>
+            <state_interface name="position"/>
+            <state_interface name="velocity"/>
+        </joint>
+    </ros2_control>
+    <gazebo>
+        <plugin name="gazebo_ros2_control" filename="libgazebo_ros2_control.so">
+            <parameters>$(find synhive_robot)/config/my_controllers.yaml</parameters>
+        </plugin>
+    </gazebo>
 </robot>
