Commit message: real robot done sim no

File: description/ros2_control.xacro (robot description, xacro)
@@ -1,9 +1,53 @@
 <?xml version="1.0"?>
 <robot xmlns:xacro="http://www.ros.org/wiki/xacro">
-    <ros2_control name="GazeboSystem" type="system">
+    <ros2_control name="FakeRobot" type="system"><!-- RealRobot -->
+        <hardware>
+            <plugin>fake_components/GenericSystem</plugin><!-- diffdrive_arduino/DiffDriveArduinoHardware  -->
+            <param name="left_wheel_names">front_left_wheel_joint,rear_left_wheel_joint</param>
+            <param name="right_wheel_names">front_right_wheel_joint,rear_right_wheel_joint</param>
+            <param name="loop_rate">30</param>
+            <param name="device">/dev/ttyUSB0</param>
+            <param name="baud_rate">57600</param>
+            <param name="timeout_ms">1000</param>
+            <param name="enc_counts_per_rev">3436</param>
+        </hardware>
+        <!-- Define all 4 wheel joints -->
+        <joint name="front_left_wheel_joint">
+            <command_interface name="velocity">
+                <param name="min">-10</param>
+                <param name="max">10</param>
+            </command_interface>
+    <state_interface name="position" />
+    <state_interface name="velocity" />
+        </joint>
+        <joint name="rear_left_wheel_joint">
+            <command_interface name="velocity">
+                <param name="min">-10</param>
+                <param name="max">10</param>
+            </command_interface>
+    <state_interface name="position" />
+    <state_interface name="velocity" />
+        </joint>
+        <joint name="front_right_wheel_joint">
+            <command_interface name="velocity">
+                <param name="min">-10</param>
+                <param name="max">10</param>
+            </command_interface>
+    <state_interface name="position" />
+    <state_interface name="velocity" />
+        </joint>
+        <joint name="rear_right_wheel_joint">
+            <command_interface name="velocity">
+                <param name="min">-10</param>
+                <param name="max">10</param>
+            </command_interface>
+    <state_interface name="position" />
+    <state_interface name="velocity" />
+        </joint>
+    </ros2_control>
+    <!-- <ros2_control name="GazeboSystem" type="system">
         <hardware>
             <plugin>gazebo_ros2_control/GazeboSystem</plugin>
         </hardware>
-        <!-- Add all 4 wheel joints -->
         <joint name="front_left_wheel_joint">
             <command_interface name="velocity">
@@ -38,5 +82,5 @@
             <state_interface name="velocity"/>
         </joint>
-    </ros2_control>
+    </ros2_control> -->
     <gazebo>
         <plugin name="gazebo_ros2_control" filename="libgazebo_ros2_control.so">
